File: KiCad-Template.kicad_pcb (KiCad board)
At the start: 4 copper layers, 48.1 x 23.8 mm, 1 part, among them U1 ESP32-S3-WROOM-1

Commit message: Add PWR and GND Net Classes
Connections:
- net Net-(U1-GND-Pad1) renamed GND
- U1 pad 2: unconnected-(U1-3V3-Pad2) -> +3V3
Changed lines of the file:
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@@
 	(net 4 "unconnected-(U1-IO48-Pad25)")
 	(net 5 "unconnected-(U1-IO10-Pad18)")
-	(net 6 "Net-(U1-GND-Pad1)")
+	(net 6 "GND")
 	(net 7 "unconnected-(U1-IO17-Pad10)")
 	(net 8 "unconnected-(U1-IO14-Pad22)")
@@
 	(net 32 "unconnected-(U1-IO47-Pad24)")
 	(net 33 "unconnected-(U1-IO39-Pad32)")
-	(net 34 "unconnected-(U1-3V3-Pad2)")
+	(net 34 "+3V3")
 	(net 35 "unconnected-(U1-IO18-Pad11)")
 	(net 36 "unconnected-(U1-IO1-Pad39)")
@@
 			(size 1.5 0.9)
 			(layers "F.Cu" "F.Mask" "F.Paste")
-			(net 6 "Net-(U1-GND-Pad1)")
+			(net 6 "GND")
 			(pinfunction "GND")
 			(pintype "power_in")
@@
 			(size 1.5 0.9)
 			(layers "F.Cu" "F.Mask" "F.Paste")
-			(net 34 "unconnected-(U1-3V3-Pad2)")
+			(net 34 "+3V3")
 			(pinfunction "3V3")
 			(pintype "power_in")
@@
 			(size 1.5 0.9)
 			(layers "F.Cu" "F.Mask" "F.Paste")
-			(net 6 "Net-(U1-GND-Pad1)")
+			(net 6 "GND")
 			(pinfunction "GND")
 			(pintype "passive")
@@
 			(property pad_prop_heatsink)
 			(layers "F.Cu" "F.Mask")
-			(net 6 "Net-(U1-GND-Pad1)")
+			(net 6 "GND")
 			(pinfunction "GND")
 			(pintype "passive")
