File: KiCad-Template.kicad_pcb (KiCad board)
At the start: 4 copper layers, 48.1 x 23.8 mm, 1 part, among them U1 ESP32-S3-WROOM-1

Commit message: Update work sheet
Parts:
- removed U1: ESP32-S3-WROOM-1, Custom:ESP32-S3-WROOM-1
Other:
- board outline removed
